Commit message: Added collision

File: urdf/crab_model.urdf (robot description, URDF)
Before this commit: robot crab, 32 links, 31 joints
Links:
- link base_link: mass None -> 15
- link coxa_l1: geometry collision box size=0.16499999999999998 0.16499999999999998 0.16499999999999998; visual box size=0.16499999999999998 0.16499999999999998 0.16499999999999998
- link coxa_l2: geometry collision box size=0.16499999999999998 0.16499999999999998 0.16499999999999998; visual box size=0.16499999999999998 0.16499999999999998 0.16499999999999998
- link coxa_l3: geometry collision box size=0.16499999999999998 0.16499999999999998 0.16499999999999998; visual box size=0.16499999999999998 0.16499999999999998 0.16499999999999998
- link coxa_r1: geometry collision box size=0.16499999999999998 0.16499999999999998 0.16499999999999998; visual box size=0.16499999999999998 0.16499999999999998 0.16499999999999998
- link coxa_r2: geometry collision box size=0.16499999999999998 0.16499999999999998 0.16499999999999998; visual box size=0.16499999999999998 0.16499999999999998 0.16499999999999998
- link coxa_r3: geometry collision box size=0.16499999999999998 0.16499999999999998 0.16499999999999998; visual box size=0.16499999999999998 0.16499999999999998 0.16499999999999998
- link femur_l1: geometry collision box size=0.35 0.075 0.02; visual box size=0.35 0.075 0.02
- link femur_l2: geometry collision box size=0.35 0.075 0.02; visual box size=0.35 0.075 0.02
- link femur_l3: geometry collision box size=0.35 0.075 0.02; visual box size=0.35 0.075 0.02
- link femur_r1: geometry collision box size=0.35 0.075 0.02; visual box size=0.35 0.075 0.02
- link femur_r2: geometry collision box size=0.35 0.075 0.02; visual box size=0.35 0.075 0.02
- link femur_r3: geometry collision box size=0.35 0.075 0.02; visual box size=0.35 0.075 0.02
- link leg_center_l1: mass None -> 1
- link leg_center_l2: mass None -> 1
- link leg_center_l3: mass None -> 1
- link leg_center_r1: mass None -> 1
- link leg_center_r2: mass None -> 1
- link leg_center_r3: mass None -> 1
- link thorax: geometry collision box size=0.775 0.65 0.225; visual box size=0.775 0.65 0.225
- link tibia_l1: geometry collision box size=0.45 0.1 0.025; visual box size=0.45 0.1 0.025
- link tibia_l2: geometry collision box size=0.45 0.1 0.025; visual box size=0.45 0.1 0.025
- link tibia_l3: geometry collision box size=0.45 0.1 0.025; visual box size=0.45 0.1 0.025
- link tibia_r1: geometry collision box size=0.45 0.1 0.025; visual box size=0.45 0.1 0.025
- link tibia_r2: geometry collision box size=0.45 0.1 0.025; visual box size=0.45 0.1 0.025
- link tibia_r3: geometry collision box size=0.45 0.1 0.025; visual box size=0.45 0.1 0.025

File: urdf/crab_model.xacro (robot description, xacro)
@@ -40,5 +40,5 @@
 			</geometry>
 		</collision>
-		<!-- <xacro:box_inertia m="15" w="${base_width}" d="${base_length}" h="${base_height}" /> -->
+		<xacro:box_inertia m="15" w="${base_width}" d="${base_length}" h="${base_height}" />
 	</link>
 	<!-- Robot Footprint -->
@@ -62,4 +62,14 @@
 			</material>
 		</visual>
+		<collision>
+			<origin xyz="0 0 0" rpy="0 0 0" />
+			<geometry>
+				<box size="${15.5/20} ${13/20} ${4.5/20}" />
+				<!-- <mesh filename="package://crab_description/meshes/thorax.STL" /> -->
+			</geometry>
+			<material name="grey">
+				<color rgba="0.5 0.5 0.5 1" />
+			</material>
+		</collision>
 		<!-- <collision>
 			<geometry>
@@ -86,4 +96,5 @@
 		</joint>
 		<link name="leg_center_${side}${num}" >
+			<xacro:box_inertia m="1" w="${2/norm}" d="${9/norm}" h="${0.5/norm}" />
 		</link>
 		<joint name="coxa_joint_${side}${num}" type="revolute">
@@ -111,4 +122,19 @@
 				</material>
 			</visual>
+			<collision>
+				<xacro:if value="${side == 'l'}">
+				<origin xyz="${0.8/norm} ${0.5/norm} 0" rpy="0 0 0" />
+			</xacro:if>
+			<xacro:if value="${side == 'r'}">
+				<origin xyz="${0.8/norm} -${0.5/norm} 0" rpy="0 0 0" />
+			</xacro:if>
+				<geometry>
+					<box size="${3.3/norm} ${3.3/norm} ${3.3/norm}" />
+					<!-- <mesh filename="package://crab_description/meshes/coxa_${side}.STL" /> -->
+				</geometry>
+				<material name="">
+					<color rgba="0.7 0.7 0 1" />
+				</material>
+			</collision>
 			<!-- <collision>
 				<geometry>
@@ -137,4 +163,14 @@
 				</material>
 			</visual>
+			<collision>
+				<origin xyz="${(7/2)/norm} 0 0" rpy="0 0 0" />
+				<geometry>
+					<box size="${7/norm} ${1.5/norm} ${0.4/norm}" />
+					<!-- <mesh filename="package://crab_description/meshes/femur_${side}.STL" /> -->
+				</geometry>
+				<material name="">
+					<color rgba="0 0.7 0.7 1" />
+				</material>
+			</collision>
 			<xacro:box_inertia m="1" w="${1.5/norm}" d="${7/norm}" h="${0.4/norm}" />
 		</link>
@@ -158,4 +194,14 @@
 				</material>
 			</visual>
+			<collision>
+				<origin xyz="${((9-1.4)/2)/norm} 0 ${2/norm}" rpy="0 0 0.06" />
+				<geometry>
+					<box size="${9/norm} ${2/norm} ${0.5/norm}" />
+					<!-- <mesh filename="package://crab_description/meshes/tibia_${side}.STL" /> -->
+				</geometry>
+				<material name="">
+					<color rgba="0.7 0 0.7 1" />
+				</material>
+			</collision>
 			<!-- TODO CHECK INERTIA ORDER!!!! -->
 			<xacro:box_inertia m="1" w="${2/norm}" d="${9/norm}" h="${0.5/norm}" />
