Commit message: Fixed training to run

File: src/urdf_demo/urdf/crab_model.xacro (robot description, xacro)
@@ -252,3 +252,48 @@
 		<self_collide>1</self_collide>
     </gazebo>
+	  <!-- Contact Sensor -->
+    <gazebo reference="base_link">
+        <material>Gazebo/Blue</material>
+        <kp>1000.0</kp>
+        <kd>1000.0</kd>
+        <mu1>1000000.0</mu1>
+        <mu2>1000000.0</mu2>
+        <sensor name="contactsensor_sensor" type="contact">
+          <always_on>true</always_on>
+          <contact>
+            <collision>lowerleg_fixed_joint_lump__contactsensor_link_collision_1</collision>
+          </contact>
+          <plugin name="bumper0_plugin" filename="libgazebo_ros_bumper.so">
+            <bumperTopicName>contactsensor_state</bumperTopicName>
+            <frameName>contactsensor_link</frameName>
+          </plugin>
+        </sensor>
+    </gazebo>
+<!-- ODOM sensor -->
+	 <gazebo>
+        <plugin name="p3d_base_controller" filename="libgazebo_ros_p3d.so">
+            <alwaysOn>true</alwaysOn>
+            <!--<updateRate>50.0</updateRate>-->
+            <bodyName>base_link</bodyName>
+            <topicName>odom</topicName>
+            <gaussianNoise>0.01</gaussianNoise>
+            <frameName>world</frameName>
+            <xyzOffsets>0 0 0</xyzOffsets>
+            <rpyOffsets>0 0 0</rpyOffsets>
+        </plugin>
+    </gazebo>
+	<!-- IMU sensor -->
+	 <gazebo>
+        <plugin name="gazebo_ros_imu_controller" filename="libgazebo_ros_imu.so">
+          <robotNamespace>/hexapod</robotNamespace>
+          <topicName>imu/data</topicName>
+          <serviceName>imu/service</serviceName>
+          <bodyName>base_link</bodyName>
+          <gaussianNoise>0</gaussianNoise>
+          <rpyOffsets>0 0 0</rpyOffsets>
+          <!--<updateRate>50.0</updateRate>-->
+          <alwaysOn>true</alwaysOn>
+          <gaussianNoise>0</gaussianNoise>
+        </plugin>
+    </gazebo>
 </robot>

Commit message: Backup

File: src/urdf_demo/urdf/crab_model.xacro (robot description, xacro)
@@ -76,5 +76,5 @@
 			</geometry>
 		</collision> -->
-		<xacro:box_inertia m="0.1" w="${15.5/norm}" d="${13/norm}" h="${4.5/norm}" />
+		<xacro:box_inertia m="0.01" w="${15.5/norm}" d="${13/norm}" h="${4.5/norm}" />
 	</link>
 	<!-- Pi parameter -->
@@ -254,9 +254,9 @@
 	  <!-- Contact Sensor -->
     <gazebo reference="base_link">
-        <material>Gazebo/Blue</material>
+        <!-- <material>Gazebo/Blue</material>
         <kp>1000.0</kp>
         <kd>1000.0</kd>
         <mu1>1000000.0</mu1>
-        <mu2>1000000.0</mu2>
+        <mu2>1000000.0</mu2> -->
         <sensor name="contactsensor_sensor" type="contact">
           <always_on>true</always_on>

Commit message: Fixed rotating on itself

File: src/urdf_demo/urdf/crab_model.xacro (robot description, xacro)
@@ -223,4 +223,12 @@
 					<!-- <mesh filename="package://crab_description/meshes/tibia_${side}.STL" /> -->
 				</geometry>
+				<surface>
+					<friction>
+					<ode>
+						<mu>10000.01</mu>
+						<mu2>10000.01</mu2>
+					</ode>
+					</friction>
+				</surface>
 				<material name="">
 					<color rgba="0.7 0 0.7 1" />
@@ -254,9 +262,9 @@
 	  <!-- Contact Sensor -->
     <gazebo reference="base_link">
-        <!-- <material>Gazebo/Blue</material>
+        <material>Gazebo/Blue</material>
         <kp>1000.0</kp>
         <kd>1000.0</kd>
         <mu1>1000000.0</mu1>
-        <mu2>1000000.0</mu2> -->
+        <mu2>1000000.0</mu2>
         <sensor name="contactsensor_sensor" type="contact">
           <always_on>true</always_on>
@@ -297,3 +305,18 @@
         </plugin>
     </gazebo>
+	<xacro:macro name="friction_set" params="side num">
+		<gazebo reference="femur_${side}${num}">
+			<mu1>10000.9</mu1>
+			<mu2>10000.9</mu2>
+			<minDepth>0.001</minDepth>
+			<kp>100000000</kp>
+			<kd>1</kd>
+		</gazebo>
+	</xacro:macro>
+<xacro:friction_set side="l" num="1"/>
+<xacro:friction_set side="l" num="2" />
+<xacro:friction_set side="l" num="3" />
+<xacro:friction_set side="r" num="1" />
+<xacro:friction_set side="r" num="2" />
+<xacro:friction_set side="r" num="3" />
 </robot>

Commit message: Fixed contact sensor naming

File: src/urdf_demo/urdf/crab_model.xacro (robot description, xacro)
@@ -270,5 +270,5 @@
           <always_on>true</always_on>
           <contact>
-            <collision>lowerleg_fixed_joint_lump__contactsensor_link_collision_1</collision>
+            <collision>base_link_fixed_joint_lump__thorax_collision_1</collision>
           </contact>
           <plugin name="bumper0_plugin" filename="libgazebo_ros_bumper.so">

Commit message: Fixed inertia

File: src/urdf_demo/urdf/crab_model.xacro (robot description, xacro)
@@ -16,4 +16,13 @@
 			<inertia ixx="${(m/12) * (h*h + d*d)}" ixy="0.0" ixz="0.0" iyy="${(m/12) * (w*w + d*d)}"
 				iyz="0.0" izz="${(m/12) * (w*w + h*h)}" />
+		</inertial>
+	</xacro:macro>
+<!-- parallel axis theorem -->
+	<xacro:macro name="box_inertia_parallel_w" params="m w h d">
+		<inertial>
+			<origin xyz="0 0 0" rpy="${pi/2} 0 ${pi/2}" />
+			<mass value="${m}" />
+			<inertia ixx="${(m/12) * (h*h + d*d + w*w/4)}" ixy="0.0" ixz="0.0" iyy="${(m/12) * (w*w + d*d + w*w/4)}"
+				iyz="0.0" izz="${(m/12) * (w*w + h*h + w*w/4)}" />
 		</inertial>
 	</xacro:macro>
@@ -76,5 +85,5 @@
 			</geometry>
 		</collision> -->
-		<xacro:box_inertia m="0.03" w="${15.5/norm}" d="${13/norm}" h="${4.5/norm}" />
+		<xacro:box_inertia m="0.03" w="${13/norm}" d="${15.5/norm}" h="${4.5/norm}" />
 	</link>
 	<!-- Pi parameter -->
@@ -186,5 +195,5 @@
 				</material>
 			</collision>
-			<xacro:box_inertia m="0.01" w="${7/norm}" d="${1.5/norm}" h="${0.4/norm}" />
+			<xacro:box_inertia_parallel_w m="0.01" w="${7/norm}" d="${0.4/norm}" h="${1.5/norm}" />
 		</link>
 		<joint name="tibia_joint_${side}${num}" type="revolute">
@@ -236,5 +245,5 @@
 			</collision>
 			<!-- TODO CHECK INERTIA ORDER!!!! -->
-			<xacro:box_inertia m="0.01" w="${9/norm}" d="${2/norm}" h="${0.5/norm}" />
+			<xacro:box_inertia_parallel_w m="0.01" w="${9/norm}" d="${0.5/norm}" h="${2/norm}" />
 		</link>
 		<joint name="tibia_foot_joint_${side}${num}" type="fixed">

Commit message: Added more observations and fixed robot size

File: src/urdf_demo/urdf/crab_model.xacro (robot description, xacro)
@@ -5,5 +5,5 @@
 	<xacro:property name="base_length" value="0.42" />
 	<xacro:property name="base_height" value="0.18" /> -->
-	<xacro:property name="norm" value="20" />
+	<xacro:property name="norm" value="100" />
 	<xacro:property name="base_width" value="${13/norm}" />
 	<xacro:property name="base_length" value="${15.5/norm}" />

Commit message: Added plotting

File: src/urdf_demo/urdf/crab_model.xacro (robot description, xacro)
@@ -92,6 +92,6 @@
 	<xacro:property name="joint_lower_limit" value="-${1.5}" />
 	<xacro:property name="joint_upper_limit" value="${1.5}" />
-	<xacro:property name="joint_effort" value="10000" />
-	<xacro:property name="joint_velocity" value="100" />
+	<xacro:property name="joint_effort" value="0.2745862" />
+	<xacro:property name="joint_velocity" value="0.000031998" />
 	<!-- Leg macros -->
 	<xacro:macro name="leg" params="side num x y angle">

Commit message: Fixed inertias

File: src/urdf_demo/urdf/crab_model.xacro (robot description, xacro)
@@ -5,4 +5,5 @@
 	<xacro:property name="base_length" value="0.42" />
 	<xacro:property name="base_height" value="0.18" /> -->
+	<!-- INERTIA COORDINATE SYSTEM IS DIFFRENT THAN GAZEBO, INERTIA Y IS UP, GAZEBO Z IS UP -->
 	<xacro:property name="norm" value="100" />
 	<xacro:property name="base_width" value="${13/norm}" />
@@ -10,7 +11,7 @@
 	<xacro:property name="base_height" value="${4.5/norm}" />
 	<!-- Define macros for inertia  -->
-	<xacro:macro name="box_inertia" params="m w h d">
+	<xacro:macro name="box_inertia" params="m w h d origin_xyz rpy_x rpy_y rpy_z">
 		<inertial>
-			<origin xyz="0 0 0" rpy="${pi/2} 0 ${pi/2}" />
+			<origin xyz="${origin_xyz}" rpy="${rpy_x} ${rpy_y} ${rpy_z}"/>
 			<mass value="${m}" />
 			<inertia ixx="${(m/12) * (h*h + d*d)}" ixy="0.0" ixz="0.0" iyy="${(m/12) * (w*w + d*d)}"
@@ -19,7 +20,7 @@
 	</xacro:macro>
 <!-- parallel axis theorem -->
-	<xacro:macro name="box_inertia_parallel_w" params="m w h d">
+	<xacro:macro name="box_inertia_parallel_w" params="m w h d origin_xyz rpy_x rpy_y rpy_z">
 		<inertial>
-			<origin xyz="0 0 0" rpy="${pi/2} 0 ${pi/2}" />
+			<origin xyz="${origin_xyz}" rpy="${rpy_x} ${rpy_y} ${rpy_z}" />
 			<mass value="${m}" />
 			<inertia ixx="${(m/12) * (h*h + d*d + w*w/4)}" ixy="0.0" ixz="0.0" iyy="${(m/12) * (w*w + d*d + w*w/4)}"
@@ -63,6 +64,5 @@
 			<origin xyz="0 0 0" rpy="0 0 0" />
 			<geometry>
-				<box size="${15.5/norm} ${13/norm} ${4.5/norm}" />
-				<!-- <mesh filename="package://crab_description/meshes/thorax.STL" /> -->
+				<box size="${base_length} ${base_width} ${base_height}" />
 			</geometry>
 			<material name="grey">
@@ -73,6 +73,5 @@
 			<origin xyz="0 0 0" rpy="0 0 0" />
 			<geometry>
-				<box size="${15.5/norm} ${13/norm} ${4.5/norm}" />
-				<!-- <mesh filename="package://crab_description/meshes/thorax.STL" /> -->
+				<box size="${base_length} ${base_width} ${base_height}" />
 			</geometry>
 			<material name="grey">
@@ -85,5 +84,7 @@
 			</geometry>
 		</collision> -->
-		<xacro:box_inertia m="0.03" w="${13/norm}" d="${15.5/norm}" h="${4.5/norm}" />
+		<xacro:box_inertia rpy_x="0" rpy_y="0" rpy_z="0"
+		origin_xyz="0 0 0" m="0.03"
+		 w="${15.5/norm}" h="${13/norm}" d="${4.5/norm}" />
 	</link>
 	<!-- Pi parameter -->
@@ -105,5 +106,7 @@
 		<link name="leg_center_${side}${num}" >
 		<!-- THIS IS EXTRA -->
-			<xacro:box_inertia m="0.001" w="${1/norm}" d="${1/norm}" h="${1/norm}" />
+			<xacro:box_inertia rpy_x="0" rpy_y="0" rpy_z="0"
+			  origin_xyz="${x} ${y} 0" m="0.0001"
+			   w="${1/norm}" d="${1/norm}" h="${1/norm}" />
 		</link>
 		<joint name="coxa_joint_${side}${num}" type="revolute">
@@ -127,5 +130,5 @@
 		<link name="coxa_${side}${num}">
 			<visual>
-				<xacro:if value="${side == 'l'}">
+			<xacro:if value="${side == 'l'}">
 				<origin xyz="${0.8/norm} ${0.5/norm} 0" rpy="0 0 0" />
 			</xacro:if>
@@ -141,5 +144,5 @@
 			</visual>
 			<collision>
-				<xacro:if value="${side == 'l'}">
+			<xacro:if value="${side == 'l'}">
 				<origin xyz="${0.8/norm} ${0.5/norm} 0" rpy="0 0 0" />
 			</xacro:if>
@@ -154,7 +157,17 @@
 				</material>
 			</collision>
-			<xacro:box_inertia m="0.01" w="${3.3/norm}" d="${3.3/norm}" h="${3.3/norm}" />
+			<xacro:if value="${side == 'l'}">
+					<xacro:box_inertia rpy_x="0" rpy_y="0" rpy_z="0"
+					  origin_xyz="${0.8/norm} ${0.5/norm} 0"  m="0.01"
+					   w="${3.3/norm}" d="${3.3/norm}" h="${3.3/norm}" />
+			</xacro:if>
+			<xacro:if value="${side == 'r'}">
+					<xacro:box_inertia rpy_x="0" rpy_y="0" rpy_z="0"
+					   origin_xyz="${0.8/norm} -${0.5/norm} 0"  m="0.01"
+					   w="${3.3/norm}" d="${3.3/norm}" h="${3.3/norm}" />
+			</xacro:if>
 		</link>
 		<joint name="femur_joint_${side}${num}" type="revolute">
+		<!-- TODO check maybe +pi/2 separate for left and right -->
 			<origin xyz="${1/norm} 0 -${1/norm}" rpy="-${pi/2} 0 0" />
 			<parent link="coxa_${side}${num}" />
@@ -179,5 +192,4 @@
 				<geometry>
 					<box size="${7/norm} ${1.5/norm} ${0.4/norm}" />
-					<!-- <mesh filename="package://crab_description/meshes/femur_${side}.STL" /> -->
 				</geometry>
 				<material name="">
@@ -189,5 +201,4 @@
 				<geometry>
 					<box size="${7/norm} ${1.5/norm} ${0.4/norm}" />
-					<!-- <mesh filename="package://crab_description/meshes/femur_${side}.STL" /> -->
 				</geometry>
 				<material name="">
@@ -195,5 +206,7 @@
 				</material>
 			</collision>
-			<xacro:box_inertia_parallel_w m="0.01" w="${7/norm}" d="${0.4/norm}" h="${1.5/norm}" />
+			<xacro:box_inertia_parallel_w rpy_x="0" rpy_y="0" rpy_z="0"
+			 origin_xyz="${(7/2)/norm} 0 0" m="0.01"
+			  w="${7/norm}" d="${0.4/norm}" h="${1.5/norm}" />
 		</link>
 		<joint name="tibia_joint_${side}${num}" type="revolute">
@@ -220,5 +233,4 @@
 				<geometry>
 					<box size="${9/norm} ${2/norm} ${0.5/norm}" />
-					<!-- <mesh filename="package://crab_description/meshes/tibia_${side}.STL" /> -->
 				</geometry>
 				<material name="">
@@ -230,5 +242,4 @@
 				<geometry>
 					<box size="${9/norm} ${2/norm} ${0.5/norm}" />
-					<!-- <mesh filename="package://crab_description/meshes/tibia_${side}.STL" /> -->
 				</geometry>
 				<surface>
@@ -244,6 +255,7 @@
 				</material>
 			</collision>
-			<!-- TODO CHECK INERTIA ORDER!!!! -->
-			<xacro:box_inertia_parallel_w m="0.01" w="${9/norm}" d="${0.5/norm}" h="${2/norm}" />
+			<xacro:box_inertia_parallel_w rpy_x="0" rpy_y="0" rpy_z="0.06"
+			 origin_xyz="${((9-1.4)/2)/norm} 0 ${2/norm}" m="0.01"
+			  w="${9/norm}" d="${0.5/norm}" h="${2/norm}" />
 		</link>
 		<joint name="tibia_foot_joint_${side}${num}" type="fixed">
