Commit message: Added collision to tibia in urdf

File: src/urdf_demo/urdf/crab_model.xacro (robot description, xacro)
@@ -238,5 +238,5 @@
 				</material>
 			</visual>
-			<collision>
+			<collision name='tibia_${side}${num}_collision'>
 				<origin xyz="${((9-1.4)/2)/norm} 0 ${2/norm}" rpy="0 0 0.06" />
 				<geometry>
@@ -325,19 +325,106 @@
           <gaussianNoise>0</gaussianNoise>
         </plugin>
-    </gazebo>
-	<xacro:macro name="friction_set" params="side num">
-		<gazebo reference="femur_${side}${num}">
-			<mu1>10000.9</mu1>
-			<mu2>10000.9</mu2>
-			<minDepth>0.001</minDepth>
-			<kp>100000000</kp>
-			<kd>1</kd>
-		</gazebo>
-	</xacro:macro>
-<xacro:friction_set side="l" num="1"/>
-<xacro:friction_set side="l" num="2" />
-<xacro:friction_set side="l" num="3" />
-<xacro:friction_set side="r" num="1" />
-<xacro:friction_set side="r" num="2" />
-<xacro:friction_set side="r" num="3" />
+   </gazebo>
+	    <gazebo reference="tibia_l1">
+			<material>Gazebo/Blue</material>
+			<kp>1000.0</kp>
+			<kd>1000.0</kd>
+			<mu1>1000000.0</mu1>
+			<mu2>1000000.0</mu2>
+			<sensor name="new_contactsensor_sensor" type="contact">
+				<always_on>true</always_on>
+				<contact>
+					<collision>tibia_l1_collision_collision</collision>
+				</contact>
+				<plugin name="bumper0_plugin" filename="libgazebo_ros_bumper.so">
+					<bumperTopicName>tibia_l1_collision</bumperTopicName>
+					<frameName>contactsensor_link</frameName>
+				</plugin>
+			</sensor>
+    	</gazebo>
+		   <gazebo reference="tibia_l2">
+			<material>Gazebo/Blue</material>
+			<kp>1000.0</kp>
+			<kd>1000.0</kd>
+			<mu1>1000000.0</mu1>
+			<mu2>1000000.0</mu2>
+			<sensor name="new_contactsensor_sensor" type="contact">
+				<always_on>true</always_on>
+					<contact>
+					<collision>tibia_l2_collision_collision</collision>
+				</contact>
+				<plugin name="bumper0_plugin" filename="libgazebo_ros_bumper.so">
+					<bumperTopicName>tibia_l2_collision</bumperTopicName>
+					<frameName>contactsensor_link</frameName>
+				</plugin>
+			</sensor>
+    	</gazebo>
+		   <gazebo reference="tibia_l3">
+			<material>Gazebo/Blue</material>
+			<kp>1000.0</kp>
+			<kd>1000.0</kd>
+			<mu1>1000000.0</mu1>
+			<mu2>1000000.0</mu2>
+			<sensor name="new_contactsensor_sensor" type="contact">
+				<always_on>true</always_on>
+					<contact>
+					<collision>tibia_l3_collision_collision</collision>
+				</contact>
+				<plugin name="bumper0_plugin" filename="libgazebo_ros_bumper.so">
+					<bumperTopicName>tibia_l3_collision</bumperTopicName>
+					<frameName>contactsensor_link</frameName>
+				</plugin>
+			</sensor>
+    	</gazebo>
+		   <gazebo reference="tibia_r1">
+			<material>Gazebo/Blue</material>
+			<kp>1000.0</kp>
+			<kd>1000.0</kd>
+			<mu1>1000000.0</mu1>
+			<mu2>1000000.0</mu2>
+			<sensor name="new_contactsensor_sensor" type="contact">
+				<always_on>true</always_on>
+					<contact>
+					<collision>tibia_r1_collision_collision</collision>
+				</contact>
+				<plugin name="bumper0_plugin" filename="libgazebo_ros_bumper.so">
+					<bumperTopicName>tibia_r1_collision</bumperTopicName>
+					<frameName>contactsensor_link</frameName>
+				</plugin>
+			</sensor>
+    	</gazebo>
+		   <gazebo reference="tibia_r2">
+			<material>Gazebo/Blue</material>
+			<kp>1000.0</kp>
+			<kd>1000.0</kd>
+			<mu1>1000000.0</mu1>
+			<mu2>1000000.0</mu2>
+			<sensor name="new_contactsensor_sensor" type="contact">
+				<always_on>true</always_on>
+					<contact>
+					<collision>tibia_r2_collision_collision</collision>
+				</contact>
+				<plugin name="bumper0_plugin" filename="libgazebo_ros_bumper.so">
+					<bumperTopicName>tibia_r2_collision</bumperTopicName>
+					<frameName>contactsensor_link</frameName>
+				</plugin>
+			</sensor>
+    	</gazebo>
+		   <gazebo reference="tibia_r3">
+			<material>Gazebo/Blue</material>
+			<kp>1000.0</kp>
+			<kd>1000.0</kd>
+			<mu1>1000000.0</mu1>
+			<mu2>1000000.0</mu2>
+			<sensor name="new_contactsensor_sensor" type="contact">
+				<always_on>true</always_on>
+					<contact>
+					<collision>tibia_r3_collision_collision</collision>
+				</contact>
+				<plugin name="bumper0_plugin" filename="libgazebo_ros_bumper.so">
+					<bumperTopicName>tibia_r3_collision</bumperTopicName>
+					<frameName>contactsensor_link</frameName>
+				</plugin>
+			</sensor>
+    	</gazebo>
 </robot>

File: src/urdf_demo/urdf/robot.urdf (robot description, URDF)
Before this commit: robot hexapod, 32 links, 31 joints
Links:
- link base_link: geometry collision box size=0.155 0.13 0.045
- link coxa_l1: geometry collision box size=0.033 0.033 0.033; visual box size=0.033 0.033 0.033
- link coxa_l2: geometry collision box size=0.033 0.033 0.033; visual box size=0.033 0.033 0.033
- link coxa_l3: geometry collision box size=0.033 0.033 0.033; visual box size=0.033 0.033 0.033
- link coxa_r1: geometry collision box size=0.033 0.033 0.033; visual box size=0.033 0.033 0.033
- link coxa_r2: geometry collision box size=0.033 0.033 0.033; visual box size=0.033 0.033 0.033
- link coxa_r3: geometry collision box size=0.033 0.033 0.033; visual box size=0.033 0.033 0.033
- link femur_l1: geometry collision box size=0.07 0.015 0.004; visual box size=0.07 0.015 0.004
- link femur_l2: geometry collision box size=0.07 0.015 0.004; visual box size=0.07 0.015 0.004
- link femur_l3: geometry collision box size=0.07 0.015 0.004; visual box size=0.07 0.015 0.004
- link femur_r1: geometry collision box size=0.07 0.015 0.004; visual box size=0.07 0.015 0.004
- link femur_r2: geometry collision box size=0.07 0.015 0.004; visual box size=0.07 0.015 0.004
- link femur_r3: geometry collision box size=0.07 0.015 0.004; visual box size=0.07 0.015 0.004
- link leg_center_l1: mass 0.001 -> 0.0001
- link leg_center_l2: mass 0.001 -> 0.0001
- link leg_center_l3: mass 0.001 -> 0.0001
- link leg_center_r1: mass 0.001 -> 0.0001
- link leg_center_r2: mass 0.001 -> 0.0001
- link leg_center_r3: mass 0.001 -> 0.0001
- link thorax: geometry collision box size=0.155 0.13 0.045; visual box size=0.155 0.13 0.045
- link tibia_l1: geometry collision box size=0.09 0.02 0.005; visual box size=0.09 0.02 0.005
- link tibia_l2: geometry collision box size=0.09 0.02 0.005; visual box size=0.09 0.02 0.005
- link tibia_l3: geometry collision box size=0.09 0.02 0.005; visual box size=0.09 0.02 0.005
- link tibia_r1: geometry collision box size=0.09 0.02 0.005; visual box size=0.09 0.02 0.005
- link tibia_r2: geometry collision box size=0.09 0.02 0.005; visual box size=0.09 0.02 0.005
- link tibia_r3: geometry collision box size=0.09 0.02 0.005; visual box size=0.09 0.02 0.005
Joints:
- joint coxa_joint_l1: limit lower=-1.5 upper=1.5 effort=10000 velocity=100 -> lower=-1.5 upper=1.5 effort=0.2745862 velocity=3.1998e-05
- joint coxa_joint_l2: limit lower=-1.5 upper=1.5 effort=10000 velocity=100 -> lower=-1.5 upper=1.5 effort=0.2745862 velocity=3.1998e-05
- joint coxa_joint_l3: limit lower=-1.5 upper=1.5 effort=10000 velocity=100 -> lower=-1.5 upper=1.5 effort=0.2745862 velocity=3.1998e-05
- joint coxa_joint_r1: limit lower=-1.5 upper=1.5 effort=10000 velocity=100 -> lower=-1.5 upper=1.5 effort=0.2745862 velocity=3.1998e-05
- joint coxa_joint_r2: limit lower=-1.5 upper=1.5 effort=10000 velocity=100 -> lower=-1.5 upper=1.5 effort=0.2745862 velocity=3.1998e-05
- joint coxa_joint_r3: limit lower=-1.5 upper=1.5 effort=10000 velocity=100 -> lower=-1.5 upper=1.5 effort=0.2745862 velocity=3.1998e-05
- joint femur_joint_l1: limit lower=-1.5 upper=1.5 effort=10000 velocity=100 -> lower=-1.5 upper=1.5 effort=0.2745862 velocity=3.1998e-05; origin xyz=0.05 0 -0.05 rpy=-1.5707963267948966 0 0 -> xyz=0.01 0 -0.01 rpy=-1.5707963267948966 0 0
- joint femur_joint_l2: limit lower=-1.5 upper=1.5 effort=10000 velocity=100 -> lower=-1.5 upper=1.5 effort=0.2745862 velocity=3.1998e-05; origin xyz=0.05 0 -0.05 rpy=-1.5707963267948966 0 0 -> xyz=0.01 0 -0.01 rpy=-1.5707963267948966 0 0
- joint femur_joint_l3: limit lower=-1.5 upper=1.5 effort=10000 velocity=100 -> lower=-1.5 upper=1.5 effort=0.2745862 velocity=3.1998e-05; origin xyz=0.05 0 -0.05 rpy=-1.5707963267948966 0 0 -> xyz=0.01 0 -0.01 rpy=-1.5707963267948966 0 0
- joint femur_joint_r1: limit lower=-1.5 upper=1.5 effort=10000 velocity=100 -> lower=-1.5 upper=1.5 effort=0.2745862 velocity=3.1998e-05; origin xyz=0.05 0 -0.05 rpy=-1.5707963267948966 0 0 -> xyz=0.01 0 -0.01 rpy=-1.5707963267948966 0 0
- joint femur_joint_r2: limit lower=-1.5 upper=1.5 effort=10000 velocity=100 -> lower=-1.5 upper=1.5 effort=0.2745862 velocity=3.1998e-05; origin xyz=0.05 0 -0.05 rpy=-1.5707963267948966 0 0 -> xyz=0.01 0 -0.01 rpy=-1.5707963267948966 0 0
- joint femur_joint_r3: limit lower=-1.5 upper=1.5 effort=10000 velocity=100 -> lower=-1.5 upper=1.5 effort=0.2745862 velocity=3.1998e-05; origin xyz=0.05 0 -0.05 rpy=-1.5707963267948966 0 0 -> xyz=0.01 0 -0.01 rpy=-1.5707963267948966 0 0
- joint leg_center_joint_l1: origin xyz=0.3875 0.325 0 rpy=0 0 0 -> xyz=0.0775 0.065 0 rpy=0 0 0
- joint leg_center_joint_l2: origin xyz=0 0.325 0 rpy=0 0 0 -> xyz=0 0.065 0 rpy=0 0 0
- joint leg_center_joint_l3: origin xyz=-0.3875 0.325 0 rpy=0 0 0 -> xyz=-0.0775 0.065 0 rpy=0 0 0
- joint leg_center_joint_r1: origin xyz=0.3875 -0.325 0 rpy=0 0 0 -> xyz=0.0775 -0.065 0 rpy=0 0 0
- joint leg_center_joint_r2: origin xyz=0 -0.325 0 rpy=0 0 0 -> xyz=0 -0.065 0 rpy=0 0 0
- joint leg_center_joint_r3: origin xyz=-0.3875 -0.325 0 rpy=0 0 0 -> xyz=-0.0775 -0.065 0 rpy=0 0 0
- joint tibia_joint_l1: limit lower=-1.5 upper=1.5 effort=10000 velocity=100 -> lower=-1.5 upper=1.5 effort=0.2745862 velocity=3.1998e-05; origin xyz=0.32999999999999996 0 0 rpy=3.141592653589793 0 1.5707963267948966 -> xyz=0.066 0 0 rpy=3.141592653589793 0 1.5707963267948966
- joint tibia_joint_l2: limit lower=-1.5 upper=1.5 effort=10000 velocity=100 -> lower=-1.5 upper=1.5 effort=0.2745862 velocity=3.1998e-05; origin xyz=0.32999999999999996 0 0 rpy=3.141592653589793 0 1.5707963267948966 -> xyz=0.066 0 0 rpy=3.141592653589793 0 1.5707963267948966
- joint tibia_joint_l3: limit lower=-1.5 upper=1.5 effort=10000 velocity=100 -> lower=-1.5 upper=1.5 effort=0.2745862 velocity=3.1998e-05; origin xyz=0.32999999999999996 0 0 rpy=3.141592653589793 0 1.5707963267948966 -> xyz=0.066 0 0 rpy=3.141592653589793 0 1.5707963267948966
- joint tibia_joint_r1: limit lower=-1.5 upper=1.5 effort=10000 velocity=100 -> lower=-1.5 upper=1.5 effort=0.2745862 velocity=3.1998e-05; origin xyz=0.32999999999999996 0 0 rpy=3.141592653589793 0 1.5707963267948966 -> xyz=0.066 0 0 rpy=3.141592653589793 0 1.5707963267948966
- joint tibia_joint_r2: limit lower=-1.5 upper=1.5 effort=10000 velocity=100 -> lower=-1.5 upper=1.5 effort=0.2745862 velocity=3.1998e-05; origin xyz=0.32999999999999996 0 0 rpy=3.141592653589793 0 1.5707963267948966 -> xyz=0.066 0 0 rpy=3.141592653589793 0 1.5707963267948966
- joint tibia_joint_r3: limit lower=-1.5 upper=1.5 effort=10000 velocity=100 -> lower=-1.5 upper=1.5 effort=0.2745862 velocity=3.1998e-05; origin xyz=0.32999999999999996 0 0 rpy=3.141592653589793 0 1.5707963267948966 -> xyz=0.066 0 0 rpy=3.141592653589793 0 1.5707963267948966

Commit message: Patched tibia sensors

File: src/urdf_demo/urdf/crab_model.xacro (robot description, xacro)
@@ -260,9 +260,27 @@
 		</link>
 		<joint name="tibia_foot_joint_${side}${num}" type="fixed">
-			<origin xyz="0.117 0 0" rpy="0 0 0" />
+			<origin xyz="${((9-1.4)/2)/norm} 0 0" rpy="0 0 0" />
 			<parent link="tibia_${side}${num}" />
 			<child link="tibia_foot_${side}${num}" />
 		</joint>
-		<link name="tibia_foot_${side}${num}" />
+		<link name="tibia_foot_${side}${num}">
+			<collision name='tibia_foot${side}${num}_collision'>
+				<origin xyz="0 0 0" rpy="0 0 0" />
+				<geometry>
+					<box size="${0.01/norm} ${0.01/norm} ${0.01/norm}" />
+				</geometry>
+				<surface>
+					<friction>
+					<ode>
+						<mu>10000.01</mu>
+						<mu2>10000.01</mu2>
+					</ode>
+					</friction>
+				</surface>
+				<material name="">
+					<color rgba="0.7 0 0.7 1" />
+				</material>
+			</collision>
+		</link>
 	</xacro:macro>
 	<xacro:property name="x_far_offset" value="${(15.5/2)/norm}" />
@@ -326,5 +344,5 @@
         </plugin>
    </gazebo>
-	    <gazebo reference="tibia_l1">
+	    <gazebo reference="tibia_foot_l1">
 			<material>Gazebo/Blue</material>
 			<kp>1000.0</kp>
@@ -335,5 +353,5 @@
 				<always_on>true</always_on>
 				<contact>
-					<collision>tibia_l1_collision_collision</collision>
+					<collision>tibia_foot_l1_collision_collision</collision>
 				</contact>
 				<plugin name="bumper0_plugin" filename="libgazebo_ros_bumper.so">
@@ -343,5 +361,5 @@
 			</sensor>
     	</gazebo>
-		   <gazebo reference="tibia_l2">
+		   <gazebo reference="tibia_foot_l2">
 			<material>Gazebo/Blue</material>
 			<kp>1000.0</kp>
@@ -352,5 +370,5 @@
 				<always_on>true</always_on>
 					<contact>
-					<collision>tibia_l2_collision_collision</collision>
+					<collision>tibia_foot_l2_collision_collision</collision>
 				</contact>
 				<plugin name="bumper0_plugin" filename="libgazebo_ros_bumper.so">
@@ -360,5 +378,5 @@
 			</sensor>
     	</gazebo>
-		   <gazebo reference="tibia_l3">
+		   <gazebo reference="tibia_foot_l3">
 			<material>Gazebo/Blue</material>
 			<kp>1000.0</kp>
@@ -369,5 +387,5 @@
 				<always_on>true</always_on>
 					<contact>
-					<collision>tibia_l3_collision_collision</collision>
+					<collision>tibia_foot_l3_collision_collision</collision>
 				</contact>
 				<plugin name="bumper0_plugin" filename="libgazebo_ros_bumper.so">
@@ -377,5 +395,5 @@
 			</sensor>
     	</gazebo>
-		   <gazebo reference="tibia_r1">
+		   <gazebo reference="tibia_foot_r1">
 			<material>Gazebo/Blue</material>
 			<kp>1000.0</kp>
@@ -386,5 +404,5 @@
 				<always_on>true</always_on>
 					<contact>
-					<collision>tibia_r1_collision_collision</collision>
+					<collision>tibia_foot_r1_collision_collision</collision>
 				</contact>
 				<plugin name="bumper0_plugin" filename="libgazebo_ros_bumper.so">
@@ -394,5 +412,5 @@
 			</sensor>
     	</gazebo>
-		   <gazebo reference="tibia_r2">
+		   <gazebo reference="tibia_foot_r2">
 			<material>Gazebo/Blue</material>
 			<kp>1000.0</kp>
@@ -403,5 +421,5 @@
 				<always_on>true</always_on>
 					<contact>
-					<collision>tibia_r2_collision_collision</collision>
+					<collision>tibia_foot_r2_collision_collision</collision>
 				</contact>
 				<plugin name="bumper0_plugin" filename="libgazebo_ros_bumper.so">
@@ -411,5 +429,5 @@
 			</sensor>
     	</gazebo>
-		   <gazebo reference="tibia_r3">
+		   <gazebo reference="tibia_foot_r3">
 			<material>Gazebo/Blue</material>
 			<kp>1000.0</kp>
@@ -420,5 +438,5 @@
 				<always_on>true</always_on>
 					<contact>
-					<collision>tibia_r3_collision_collision</collision>
+					<collision>tibia_foot_r3_collision_collision</collision>
 				</contact>
 				<plugin name="bumper0_plugin" filename="libgazebo_ros_bumper.so">
